File: source/esr_tester/esr_tester.sch (KiCad schematic (older format))
At the start: 40 parts, among them IC1- TL084, J1 Conn_01x01, J2 Conn_01x01

Commit message: fix schematic, add *cache.lib file
- made visible components values
- fixed C3 value
- other small changes
Parts:
- BT?: value Battery -> 9V
- C1, C2: value 1µF elettrolitico -> 1uF
- C3: value 1pF poliestere -> 1nF; Type (none) -> Polyester
- C4: value 100000 pF poliestere -> 100nF; Type (none) -> Polyester
- C5, C6: value 1µF poliestere -> 1uF; Type (none) -> Polyester
- J1, J2: symbol Conn_01x01 -> CONN_01X01
- R11, R9: value 1k 1% -> 1k; Tolerance (none) -> 1%
Connections:
- net labels added: +4.5V, -4.5V
- wire segments 90 -> 138
Other:
- note removed: "Corretto?"
- note removed: "Da controllare. Sulla rivista c'è \nscritto "massa fittizia""
- note removed: "Nel campo Value, è corretto scrivere "22R" per un resistore da 22 Ohm?"
- note removed: "cosa vuol dire 4.5 V ? Vedi rivista."
- moved on the sheet: TR2

Commit message: schematic annotation
Parts:
- gave numbers to parts that had none: 2
- renumbered IC1- to IC1-1
Connections:
- net at R14.1, R16.1: now also IC1-1.10 (+); no longer IC1-1.5 (+)
- net at R13.1, R15.2: now also IC1-1.9 (-); no longer IC1-1.6 (-)
- net at C4.2, R15.1, R18.2: now also IC1-1.8; no longer IC1-1.7
- net at C4.1, R17.1: now also IC1-1.12 (+); no longer IC1-1.10 (+)
- net at DS3.2 (A): now also IC1-1.14; no longer IC1-1.8
- net at C6.1, DS3.1 (K), R20.2: now also IC1-1.13 (-); no longer IC1-1.9 (-)
- net at R1.1, R3.2: now also IC1-1.5 (+); no longer IC1-1.12 (+)
- net at C3.1, R2.2: now also IC1-1.6 (-); no longer IC1-1.13 (-)
- net at R2.1, R3.1, R6.2: now also IC1-1.7; no longer IC1-1.14

Commit message: footprint association (schematics and netlist)
Parts:
- BT1: footprint (none) -> Pin_Headers:Pin_Header_Straight_1x02_Pitch2.54mm
- C1, C2: footprint (none) -> Capacitors_THT:CP_Radial_D5.0mm_P2.50mm
- C3, C4, C5, C6: footprint (none) -> Capacitors_THT:C_Disc_D3.0mm_W1.6mm_P2.50mm
- DL1: footprint (none) -> LEDs:LED_D3.0mm
- DS1, DS2, DS3: footprint (none) -> Diodes_THT:D_5W_P5.08mm_Vertical_AnodeUp
- IC1-1: footprint (none) -> Housings_DIP:DIP-14_W7.62mm
- J1, J2: footprint (none) -> Connectors:Banana_Jack_1Pin
- MES1: footprint (none) -> Connectors:Banana_Jack_2Pin
- R1, R10, R11, R12, R13, R14, R15, R16, R17, R18, R19, R2, R20, R3, R4, R5, R6, R7, R8, R9: footprint (none) -> Resistors_THT:R_Axial_DIN0204_L3.6mm_D1.6mm_P5.08mm_Horizontal
- R21: footprint (none) -> Potentiometers:Potentiometer_Trimmer_ACP_CA9v_Horizontal_Px10.0mm_Py5.0mm
- S1: footprint (none) -> Buttons_Switches_THT:SW_PUSH-12mm

Commit message: Add a special «Power Flag» to indicate to KiCad that power comes from somewhere. This will avoid ERC warning.
Parts:
- S1: symbol SW_DIP_x01 -> SW_DIP_x01-RESCUE-esr_tester
Other:
- note added: "Add a Power Flag to \nindicate to KiCad that \npower comes from somewhere. \nThis will avoid the ERC warning."
Changed lines of the file:
@@
 $EndDescr
 $Comp
-L SW_DIP_x01 S1
+L SW_DIP_x01-RESCUE-esr_tester S1
 U 1 1 59E2A8BC
 P 850 1450
@@
 $Bitmap
 Pos 4750 6800
-Scale 1,000000
+Scale 1.000000
 Data
 89 50 4E 47 0D 0A 1A 0A 00 00 00 0D 49 48 44 52 00 00 01 48 00 00 00 F9 08 02 00 00 00 CA 97 3B
@@
 Text Notes 3000 7000 0    60   ~ 0
 Qui ci sarebbero \ni coccodrilli/puntali.
-Text Notes 7000 6350 0    118  ~ 0
+Text Notes 7000 6350 0    39   ~ 0
 Lo schema dell'integrato TL084, come \npresente nella libreria di Kicad è diverso \nda come è disegnato nella rivista. \nHo collegato come da rivista i pin \nin base al loro numero, piuttosto che \nin base alle sottounità (A,B,C,D) del IC.
 $Comp
@@
 Wire Wire Line
 	2450 2800 2450 2050
+$Comp
+L PWR_FLAG #FLG?
+U 1 1 5A2D7459
+P 9750 3150
+F 0 "#FLG?" H 9750 3225 50  0001 C CNN
+F 1 "PWR_FLAG" H 9750 3300 50  0000 C CNN
+F 2 "" H 9750 3150 50  0001 C CNN
+F 3 "" H 9750 3150 50  0001 C CNN
+	1    9750 3150
+	1    0    0    -1
+$EndComp
+$Comp
+L PWR_FLAG #FLG?
+U 1 1 5A2D74C3
+P 10400 3150
+F 0 "#FLG?" H 10400 3225 50  0001 C CNN
+F 1 "PWR_FLAG" H 10400 3300 50  0000 C CNN
+F 2 "" H 10400 3150 50  0001 C CNN
+F 3 "" H 10400 3150 50  0001 C CNN
+	1    10400 3150
+	1    0    0    -1
+$EndComp
+Wire Wire Line
+	9750 3150 9750 3300
+Wire Wire Line
+	10400 3150 10400 3350
+Text Label 9750 3300 0    60   ~ 0
++4.5V
+Text Label 10400 3350 0    60   ~ 0
+-4.5V
+Text Notes 9450 2650 0    60   ~ 0
+Add a Power Flag to \nindicate to KiCad that \npower comes from somewhere. \nThis will avoid the ERC warning.
 $EndSCHEMATC
